Commit message: Adds collision mesh for base_link.
Former-commit-id: f5181da576ffff29da6c9f3386a265fc2fb33821

File: robomagellan_description/urdf/robomagellan.urdf.xacro (robot description, xacro)
@@ -22,5 +22,5 @@
         <collision>
             <geometry>
-                <box size="0.3302 0.4445 0.0508"/>
+                <mesh filename="package://robomagellan_description/meshes/Robot_Collision.dae"/>
             </geometry>
             <origin xyz="-0.1397 0 0" rpy="0 0 0"/>

Commit message: IMU-related tweaks.
Former-commit-id: 58a4f0b71a0e9e1f9c5c2e98bf3f97131d53c89f

File: robomagellan_description/urdf/robomagellan.urdf.xacro (robot description, xacro)
@@ -10,5 +10,4 @@
         <color rgba="0 0 0 1"/>
     </material>
-    <!-- TODO consider actually modelling the caster wheel. I don't think it'd actually be that hard -->
     <xacro:include filename="$(find realsense2_description)/urdf/_d435.urdf.xacro"/>
     <link name="base_link">
@@ -40,4 +39,12 @@
             <material name="black"/>
         </visual>
+    </link>
+    <link name="imu">
+        <visual>
+            <geometry>
+                <box size="0.0381 0.0381 0.0127" />
+            </geometry>
+        </visual>
+        <material name="black"/>
     </link>
     <link name="left_wheel">
@@ -101,4 +108,9 @@
         <origin xyz="0.0508 0 0.381" rpy="0 0 0"/>
     </joint>
+    <joint name="imu_joint" type="fixed">
+        <parent link="base_link"/>
+        <child link="imu"/>
+        <origin xyz="0 0 0" rpy="0 0 0"/>
+    </joint>
     <xacro:sensor_d435 parent="base_link">
         <origin xyz="0.0762 0 0.20955" rpy="0 0 0"/>
@@ -140,4 +152,37 @@
             <robotNamespace>/</robotNamespace>
         </plugin>
+        <plugin filename="libhector_gazebo_ros_imu.so" name="imu">
+            <serviceName>/imu/calibrate</serviceName>
+            <updateRate>200.0</updateRate>
+            <bodyName>imu</bodyName>
+            <frameId>imu</frameId>
+            <topicName>/imu</topicName>
+            <rpyOffsets>0 0 0</rpyOffsets>
+            <gaussianNoise>0.00000001</gaussianNoise>
+            <accelDrift>0.00000001 0.00000001 0.00000001</accelDrift>
+            <accelDriftFrequency>0.00000001 0.00000001 0.00000001</accelDriftFrequency>
+            <accelGaussianNoise>0.00000001 0.00000001 0.00000001</accelGaussianNoise>
+            <rateDrift>0.0 0.0 0.0</rateDrift>
+            <rateDriftFrequency>0.0 0.0 0.0</rateDriftFrequency>
+            <rateGaussianNoise>0.0 0.0 0.0</rateGaussianNoise>
+            <headingDrift>0.0 0.0 0.0</headingDrift>
+            <headingDriftFrequency>0.0 0.0 0.0</headingDriftFrequency>
+            <headingGaussianNoise>0.0 0.0 0.0</headingGaussianNoise>
+            <yawOffset>1.57079632679</yawOffset>
+        </plugin>
+        <plugin filename="libhector_gazebo_ros_gps.so" name="gps">
+            <updateRate>20.0</updateRate>
+            <bodyName>base_link</bodyName>
+            <frameId>base_link</frameId>
+            <topicName>/fix</topicName>
+            <velocityTopicName>/fix_velocity</velocityTopicName>
+            <referenceLatitude>47.653150</referenceLatitude>
+            <referenceLongitude>-122.343939</referenceLongitude>
+            <referenceAltitude>30.0</referenceAltitude>
+            <drift>0.001 0.001 0.001</drift>
+            <gaussianNoise>0.0001 0.0001 0.0001</gaussianNoise>
+            <velocityDrift>0 0 0</velocityDrift>
+            <velocityGaussianNoise>0.005 0.005 0.05</velocityGaussianNoise>
+        </plugin>
     </gazebo>
 </robot>

Commit message: Tweaks towards getting localization working.
Former-commit-id: 1c0184168a85af0fe51f92e618a0fc01088507ec

File: robomagellan_description/urdf/robomagellan.urdf.xacro (robot description, xacro)
@@ -111,5 +111,5 @@
         <parent link="base_link"/>
         <child link="imu"/>
-        <origin xyz="0 0 0" rpy="0 0 0"/>
+        <origin xyz="0 0 0.1397" rpy="0 -1.57079632679 3.14159265359"/>
     </joint>
     <xacro:sensor_d435 parent="base_link">
